File: PCB/PCB-verbesserung_2025-06-02.brd (EAGLE design)
At the start: 60 x 60 mm, 16 parts

Commit message: PCB aktualisiert
Parts:
- removed QUFVJSCI: (no value), PCB-verbesserung_2025-05-29:QUFVJSCI_1PRIMARY
- added DHDYFYKT: (no value), PCB-verbesserung_2025-06-02 (2):DHDYFYKT_1PRIMARY
- 24: device PCB-verbesserung_2025-05-29:PIN-HEADER-210S-2X12P_WK_1PRIMARY -> PCB-verbesserung_2025-06-02 (2):PIN-HEADER-210S-2X12P_WK_1PRIMARY
- CCS811: device PCB-verbesserung_2025-05-29:CCS811_JOY-IT_1PRIMARY -> PCB-verbesserung_2025-06-02 (2):CCS811_JOY-IT_1PRIMARY
- D6T1A01: device PCB-verbesserung_2025-05-29:D6T1A01_1PRIMARY -> PCB-verbesserung_2025-06-02 (2):D6T1A01_1PRIMARY
- DUMMY1, DUMMY2, DUMMY3, DUMMY4: device PCB-verbesserung_2025-05-29:P:EX40Y40D201 -> PCB-verbesserung_2025-06-02 (2):P:EX40Y40D201
- DUMMY5, DUMMY6, DUMMY7, DUMMY8: device PCB-verbesserung_2025-05-29:P:EX126Y126D1261 -> PCB-verbesserung_2025-06-02 (2):P:EX126Y126D1261
- ESP32C6: device PCB-verbesserung_2025-05-29:ESP32-C6-DEV-KIT-N8_1PRIMARY -> PCB-verbesserung_2025-06-02 (2):ESP32-C6-DEV-KIT-N8_1PRIMARY
- HYT271: device PCB-verbesserung_2025-05-29:HYT271_1PRIMARY -> PCB-verbesserung_2025-06-02 (2):HYT271_1PRIMARY
- R1, R2: device PCB-verbesserung_2025-05-29:R0603_1PRIMARY -> PCB-verbesserung_2025-06-02 (2):R0603_1PRIMARY
- moved R2 0.90 mm to (88.5, 53.6)
- moved D6T1A01 0.77 mm to (95.2, 56.2)
- moved CCS811 0.68 mm to (95.2, 89.1)
- moved DUMMY1 0.64 mm to (95.2, 67.5)
- moved DUMMY2 0.64 mm to (95.2, 66.2)
- moved DUMMY3 0.64 mm to (95.2, 64.9)
- moved DUMMY4 0.64 mm to (95.2, 63.7)
- moved HYT271 0.64 mm to (95.2, 67.5)
Routing:
- net GND: track 109.0 -> 124.6 mm
- net 5V0: track 116.0 -> 121.4 mm
- net GPIO0: track 39.1 -> 35.3 mm, vias 1 -> 0
- net GPIO10: track 43.7 -> 41.0 mm
- net GPIO9: track 16.5 -> 18.3 mm
- net SCL: track 57.1 -> 58.4 mm
- net GPIO2: track 36.4 -> 35.3 mm, vias 1 -> 0
- net SDA: track 63.9 -> 64.7 mm
- net GPIO1: track 35.2 -> 35.3 mm, vias 1 -> 0
