File: PCB/PCB-neue-Widerstände_2025-07-04.PCB.brd (EAGLE design)
At the start: 60 x 60 mm, 16 parts

Commit message: neue PCB
Parts:
- removed CONAYFJX: (no value), PCB-neu_2025-06-24:CONAYFJX_1PRIMARY
- added EBYOFHXR: (no value), PCB-neue-Widerstände_2025-07-04:EBYOFHXR_1PRIMARY
- 24: device PCB-neu_2025-06-24:PIN-HEADER-210S-2X12P_WK_1PRIMARY -> PCB-neue-Widerstände_2025-07-04:PIN-HEADER-210S-2X12P_WK_1PRIMARY
- CCS811: device PCB-neu_2025-06-24:CCS811_JOY-IT_1PRIMARY -> PCB-neue-Widerstände_2025-07-04:CCS811_JOY-IT_1PRIMARY
- D6T1A01: device PCB-neu_2025-06-24:D6T1A01_1PRIMARY -> PCB-neue-Widerstände_2025-07-04:D6T1A01_1PRIMARY
- DUMMY1, DUMMY2, DUMMY3, DUMMY4: device PCB-neu_2025-06-24:P:EX40Y40D241 -> PCB-neue-Widerstände_2025-07-04:P:EX40Y40D241
- DUMMY5, DUMMY6, DUMMY7, DUMMY8: device PCB-neu_2025-06-24:P:EX126Y126D1261 -> PCB-neue-Widerstände_2025-07-04:P:EX126Y126D1261
- ESP32-C6-DEVKITC-1: device PCB-neu_2025-06-24:ESP32-C6-DEV-KIT-N8_1PRIMARY -> PCB-neue-Widerstände_2025-07-04:ESP32-C6-DEV-KIT-N8_1PRIMARY
- HYT271: device PCB-neu_2025-06-24:HYT271_1PRIMARY -> PCB-neue-Widerstände_2025-07-04:HYT271_1PRIMARY
- R1, R2: value 4,7k -> WIDERSTAND; device PCB-neu_2025-06-24:R0603_1PRIMARY -> PCB-neue-Widerstände_2025-07-04:WIDERSTAND_1PRIMARY
- moved R2 9.58 mm to (79.7, 49.3)
- moved R1 9.39 mm to (79.7, 54.1)
Connections:
- new net S$1: 24.9, ESP32-C6-DEVKITC-1.15
- new net S$2: CCS811.3, CCS811.6
- net 5V0: now also R1.1, R2.1; no longer R1.2, R2.2
- net GND: no longer 24.9, CCS811.3, CCS811.6, ESP32-C6-DEVKITC-1.15
- net SCL: now also R1.2; no longer R2.1
- net SDA: now also R2.2; no longer R1.1
Routing:
- net GND: track 101.1 -> 28.0 mm
- net S$1: track 0.00 -> 46.5 mm
- net S$2: track 0.00 -> 26.6 mm
- net 5V0: track 116.9 -> 120.1 mm
- net SCL: track 58.5 -> 56.9 mm
- net SDA: track 66.6 -> 67.8 mm, vias 4 -> 3
